Commit message: Add keyboard teleoperation example

File: real_backhoe.urdf (robot description, URDF)
Before this commit: robot real_backhoe, 6 links, 5 joints
Links:
- removed link base
- removed link boom
- removed link bucket_cylinder
- added link boom_lower, mass 200; collision box size=0.5 0.5 1.8; visual box size=0.5 0.5 1.8
- added link boom_upper, mass 182; collision box size=0.5 0.5 1.8; visual box size=0.4 0.4 1.8
- link bucket: mass 200 -> 100.0; geometry collision box size=0.5 1.0 0.4; visual box size=0.5 1.0 0.4
- link stick: mass 400 -> 156.0; geometry collision box size=0.3 0.3 1.6; visual box size=0.3 0.3 1.6
- link turret: mass 500 -> 3000.0; geometry collision box size=1.6 1.6 0.2; visual box size=1.6 1.6 0.2
Joints:
- removed joint boom_joint
- removed joint bucket_cyl_joint
- removed joint bucket_joint
- removed joint stick_joint
- removed joint turret_joint
- added joint boom_fixed_joint: type fixed, parent boom_lower, child boom_upper, origin xyz=0 0 1.8 rpy=0 0 0
- added joint boom_to_stick: type revolute, parent boom_upper, child stick, origin xyz=0 0 1.8 rpy=0 0 0, axis 0 1 0, limit lower=-1.57 upper=1.57 effort=800 velocity=3.2
- added joint stick_to_bucket: type revolute, parent stick, child bucket, origin xyz=0 0 1.6 rpy=0 0 0, axis 0 1 0, limit lower=-1.5 upper=1.5 effort=500 velocity=1.0
- added joint turret_to_boom_lower: type revolute, parent turret, child boom_lower, origin xyz=0 0 0.5 rpy=0 0 0, axis 0 1 0, limit lower=-0.4 upper=1.2 effort=1000 velocity=1.5
